Commit message: updated for zed2 for this repo

File: common_sensors/urdf/sensors/zed2.xacro (robot description, xacro)
@@ -17,10 +17,10 @@
       <visual>
         <geometry>
-          <mesh filename="package://leo_erc_description/models/ZED2.dae"/>
+          <mesh filename="package://common_sensors/meshes/sensors/ZED2.dae"/>
         </geometry>
       </visual>
       <collision>
         <geometry>
-          <mesh filename="package://leo_erc_description/models/ZED2.dae"/>
+          <mesh filename="package://common_sensors/meshes/sensors/ZED2.dae"/>
         </geometry>
       </collision>
